Commit message: Add gazebo and transmission in urdf.

File: robot_description/urdf/car.urdf.xacro (robot description, xacro)
@@ -72,5 +72,5 @@
             <parent link="base_link"/>
             <child link="${name}_front_wheel"/>
-            <origin xyz="${off_set}  ${flag*base_link_width/2} ${-(base_link_high/2)}"/>
+            <origin xyz="${off_set}  ${flag*(base_link_width+wheel_width)/2} ${-(base_link_high/2)}"/>
             <axis xyz="0 1 0"/>
         </joint>
@@ -103,5 +103,5 @@
             <parent link="base_link"/>
             <child link="${name}_behind_wheel"/>
-            <origin xyz="${-off_set}  ${flag*base_link_width/2} ${-(base_link_high/2)}"/>
+            <origin xyz="${-off_set}  ${flag*(base_link_width+wheel_width)/2} ${-(base_link_high/2)}"/>
             <axis xyz="0 1 0"/>
         </joint>
@@ -112,3 +112,24 @@
     <xacro:behind_wheel name="left" flag="1"/>
     <xacro:behind_wheel name="right" flag="-1"/>
+    <xacro:macro name="transmission_interface" params="name">
+        <transmission name="${name}_transmission">
+            <type>transmission_interface/SimpleTransmission</type>
+            <joint name="${name}">
+                <hardwareInterface>hardware_interface/VelocityJointInterface</hardwareInterface>
+            </joint>
+            <actuator name="${name}_motor">
+                <hardwareInterface>hardware_interface/VelocityJointInterface</hardwareInterface>
+                <mechanicalReduction>1</mechanicalReduction>
+            </actuator>
+        </transmission>
+    </xacro:macro>
+    <xacro:transmission_interface name="left_front_wheel2base_link"/>
+    <xacro:transmission_interface name="right_front_wheel2base_link"/>
+    <xacro:transmission_interface name="left_behind_wheel2base_link"/>
+    <xacro:transmission_interface name="right_behind_wheel2base_link"/>
+    <gazebo>
+        <plugin name="gazebo_ros_control" filename="libgazebo_ros_control.so">
+            <robotNamespace>/</robotNamespace>
+        </plugin>
+    </gazebo>
 </robot>
